Commit message: Fixed scaling issues

File: urdf/panda_arm_bat.urdf (robot description, URDF)
Before this commit: robot panda_arm_bat, 9 links, 8 joints
Links:
- added link base_box, mass 1; collision box size=0.3 0.3 0.1; visual box size=0.3 0.3 0.1
Joints:
- added joint base_to_link0: type fixed, parent base_box, child link0, origin xyz=0 0 0.1 rpy=0 0 0

Commit message: fixed merge conflict

File: urdf/panda_arm_bat.urdf (robot description, URDF)
Before this commit: robot panda_arm_bat, 10 links, 9 joints
Links:
- link base_box: geometry collision box size=0.1 0.1 0.6; visual box size=0.3 0.3 0.6
Joints:
- joint base_to_link0: origin xyz=0 0 0.1 rpy=0 0 0 -> xyz=0 0 0.6 rpy=0 0 0
