Commit message: ppo and sac

File: models/envs/panda_arm_bat.urdf (robot description, URDF)
Before this commit: robot panda_arm_bat, 10 links, 9 joints
Links:
- link base_box: geometry collision box size=0.1 0.1 0.4; visual box size=0.3 0.3 0.4
Joints:
- joint base_to_link0: origin xyz=0 0 0.1 rpy=0 0 0 -> xyz=0 0 0.4 rpy=0 0 0

File: urdf/panda_arm_bat.urdf (robot description, URDF)
Before this commit: robot panda_arm_bat, 10 links, 9 joints
Links:
- link base_box: geometry collision box size=0.1 0.1 0.4; visual box size=0.3 0.3 0.4
Joints:
- joint base_to_link0: origin xyz=0 0 0.6 rpy=0 0 0 -> xyz=0 0 0.4 rpy=0 0 0
